Commit message: Add files via upload

File: level-1/2f1t.urdf (robot description, URDF)
Before this commit: robot origins, 5 links, 4 joints
Links:
- removed link arm
- added link arm1; visual cylinder length=1 radius=0.1
- added link arm2; visual cylinder length=1 radius=0.1
Joints:
- added joint arm_to_arm: type revolute, parent arm1, child arm2, origin xyz=0 0 0, axis 0 0 1, limit lower=-0.83 upper=1.57075 effort=1000.0 velocity=0.5
- joint arm_to_palm: axis (none) -> 0 0 1; limit (none) -> lower=-0.83 upper=1.57075 effort=1000.0 velocity=0.5; origin (none) -> xyz=0 1 0; parent arm -> arm2; type fixed -> revolute
- joint palm_to_finger_1: axis 1 0 0 -> 0 0 1; origin (none) -> xyz=0 0.5 0.1
- joint palm_to_finger_2: axis 1 0 0 -> 0 0 1; origin (none) -> xyz=0 0.5 -0.1
- joint palm_to_thumb: axis 1 0 0 -> 0 -1 0; origin (none) -> xyz=0 0.25 0.2

Commit message: Add files via upload

File: level-1/2f1t.urdf (robot description, URDF)
Before this commit: robot origins, 6 links, 5 joints
Joints:
- joint arm_to_arm: limit lower=-0.83 upper=1.57075 effort=1000.0 velocity=0.5 -> lower=0 upper=2.617 effort=1000.0 velocity=0.5

Commit message: Wrist Pronation and Supination added

File: level-1/2f1t.urdf (robot description, URDF)
Before this commit: robot origins, 6 links, 5 joints
Joints:
- joint arm_to_arm: axis 0 0 1 -> 1 0 0; limit lower=0 upper=2.617 effort=1000.0 velocity=0.5 -> lower=0.0 upper=2.617 effort=1000.0 velocity=0.5
- joint arm_to_palm: axis 0 0 1 -> 0 1 0; limit lower=-0.83 upper=1.57075 effort=1000.0 velocity=0.5 -> lower=0 upper=9 effort=1000.0 velocity=0.5; origin xyz=0 1 0 -> xyz=0 1 0 rpy=1.1 1 1.25

Commit message: Add files via upload

File: level-1/2f1t.urdf (robot description, URDF)
Before this commit: robot origins, 6 links, 5 joints
Links:
- link arm1: mass None -> 10
- link arm2: mass None -> 10
- link finger_1: mass None -> 10
- link finger_2: mass None -> 10
- link palm: mass None -> 10
- link thumb: mass None -> 10
Joints:
- joint arm_to_palm: limit lower=0 upper=9 effort=1000.0 velocity=0.5 -> lower=0 upper=9 effort=1000.0 velocity=0.01
