Commit message: update

File: urdf-practice/basic_arm.urdf (robot description, URDF)
Before this commit: robot robot-arm, 0 links, 0 joints
Links:
- added link arm1, mass 10; visual cylinder length=1 radius=0.1
- added link arm2, mass 10; visual cylinder length=1 radius=0.1
- added link finger_1, mass 10; visual box size=0.1 0.4 0.1
- added link finger_2, mass 10; visual box size=0.1 0.4 0.1
- added link palm, mass 10; visual box size=0.1 0.5 0.4
- added link thumb, mass 10; visual box size=0.1 0.1 0.4
Joints:
- added joint arm_to_arm: type revolute, parent arm1, child arm2, origin xyz=0 0 0, axis 1 0 0, limit lower=0.0 upper=2.617 effort=1000.0 velocity=0.5
- added joint arm_to_palm: type revolute, parent arm2, child palm, origin xyz=0 1 0 rpy=1.1 1 1.25, axis 0 1 0, limit lower=0 upper=9 effort=1000.0 velocity=0.01
- added joint palm_to_finger_1: type revolute, parent palm, child finger_1, origin xyz=0 0.5 0.1, axis 0 0 1, limit lower=0.0 upper=1.57075 effort=1000.0 velocity=0.5
- added joint palm_to_finger_2: type revolute, parent palm, child finger_2, origin xyz=0 0.5 -0.1, axis 0 0 1, limit lower=0.0 upper=1.57075 effort=1000.0 velocity=0.5
- added joint palm_to_thumb: type revolute, parent palm, child thumb, origin xyz=0 0.25 0.2, axis 0 -1 0, limit lower=0.0 upper=1.57075 effort=1000.0 velocity=0.5
